Commit message: changing file path for mesh files

File: b1_description/xacro/b1.urdf (robot description, URDF)
Before this commit: robot b1_description, 36 links, 35 joints
Links:
- link FL_calf: geometry collision mesh filename=../meshes/calfb.dae scale=1 1 1; visual mesh filename=../meshes/calfb.dae scale=1 1 1
- link FL_hip: geometry collision mesh filename=../meshes/hipb.dae scale=1 1 1; visual mesh filename=../meshes/hipb.dae scale=1 1 1
- link FL_thigh: geometry collision mesh filename=../meshes/thighb.dae scale=1 1 1; visual mesh filename=../meshes/thighb.dae scale=1 1 1
- link FR_calf: geometry collision mesh filename=../meshes/calfb.dae scale=1 1 1; visual mesh filename=../meshes/calfb.dae scale=1 1 1
- link FR_hip: geometry collision mesh filename=../meshes/hipb.dae scale=1 1 1; visual mesh filename=../meshes/hipb.dae scale=1 1 1
- link FR_thigh: geometry collision mesh filename=../meshes/thigh_mirrorb.dae scale=1 1 1; visual mesh filename=../meshes/thigh_mirrorb.dae scale=1 1 1
- link RL_calf: geometry collision mesh filename=../meshes/calfb.dae scale=1 1 1; visual mesh filename=../meshes/calfb.dae scale=1 1 1
- link RL_hip: geometry collision mesh filename=../meshes/hipb.dae scale=1 1 1; visual mesh filename=../meshes/hipb.dae scale=1 1 1
- link RL_thigh: geometry collision mesh filename=../meshes/thighb.dae scale=1 1 1; visual mesh filename=../meshes/thighb.dae scale=1 1 1
- link RR_calf: geometry collision mesh filename=../meshes/calfb.dae scale=1 1 1; visual mesh filename=../meshes/calfb.dae scale=1 1 1
- link RR_hip: geometry collision mesh filename=../meshes/hipb.dae scale=1 1 1; visual mesh filename=../meshes/hipb.dae scale=1 1 1
- link RR_thigh: geometry collision mesh filename=../meshes/thigh_mirrorb.dae scale=1 1 1; visual mesh filename=../meshes/thigh_mirrorb.dae scale=1 1 1
- link trunk: geometry collision mesh filename=../meshes/trunkb.dae scale=1 1 1; visual mesh filename=../meshes/trunkb.dae scale=1 1 1
